Commit message: add mesh

File: swerve2/urdf/swerve2.urdf (robot description, URDF)
Before this commit: robot swerve, 9 links, 8 joints
Links:
- link base_link: mass 3.0006 -> 3.00064129669063; geometry collision mesh filename=package://swerve2/meshes/base_link.STL; visual mesh filename=package://swerve2/meshes/base_link.STL
- link steer1: mass 0.2218 -> 0.221804775243313; geometry collision mesh filename=package://swerve2/meshes/steer1.STL; visual mesh filename=package://swerve2/meshes/steer1.STL
- link steer2: geometry collision mesh filename=package://swerve2/meshes/steer2.STL; visual mesh filename=package://swerve2/meshes/steer2.STL
- link steer3: mass 0.2218 -> 0.221804775243313; geometry collision mesh filename=package://swerve2/meshes/steer3.STL; visual mesh filename=package://swerve2/meshes/steer3.STL
- link steer4: geometry collision mesh filename=package://swerve2/meshes/steer4.STL; visual mesh filename=package://swerve2/meshes/steer4.STL
- link wheel1: mass 0.76476 -> 0.764764182848667; geometry collision mesh filename=package://swerve2/meshes/wheel1.STL; visual mesh filename=package://swerve2/meshes/wheel1.STL
- link wheel2: geometry collision mesh filename=package://swerve2/meshes/wheel2.STL; visual mesh filename=package://swerve2/meshes/wheel2.STL
- link wheel3: mass 0.76476 -> 0.764764182848667; geometry collision mesh filename=package://swerve2/meshes/wheel3.STL; visual mesh filename=package://swerve2/meshes/wheel3.STL
- link wheel4: geometry collision mesh filename=package://swerve2/meshes/wheel4.STL; visual mesh filename=package://swerve2/meshes/wheel4.STL
Joints:
- joint wheel1: origin xyz=0 0 0.015 rpy=-1.5708 -0.77448 -3.1416 -> xyz=0 0 0.015 rpy=-1.5707963267949 -0.774484498120501 -3.14159265358979
- joint wheel2: origin xyz=0.01 0 0 rpy=-1.5708 1.3789 3.1416 -> xyz=0.00999999999999995 0 0 rpy=-1.57079632679491 1.37893541128008 3.14159265358978
- joint wheel3: origin xyz=0 0 0.015 rpy=1.5708 1.5498 0 -> xyz=0 0 0.0150000000000001 rpy=1.57079632679486 1.54977467859669 0
- joint wheel4: origin xyz=0 0 0.015 rpy=-1.5708 1.0915 -3.1416 -> xyz=0 0 0.015 rpy=-1.5707963267949 1.09151535378322 -3.14159265358979
