Commit message: a

File: AiRobotURDF.SLDASM.urdf (robot description, URDF)
Before this commit: robot swerve2, 9 links, 8 joints
Links:
- removed link steer1
- removed link steer2
- removed link steer3
- removed link steer4
- removed link wheel1
- removed link wheel2
- removed link wheel3
- removed link wheel4
- added link steerBL, mass 0.98656895809198; collision mesh filename=package://AiRobotURDF.SLDASM/meshes/steerBL.STL; visual mesh filename=package://AiRobotURDF.SLDASM/meshes/steerBL.STL
- added link steerBR, mass 0.98656895809198; collision mesh filename=package://AiRobotURDF.SLDASM/meshes/steerBR.STL; visual mesh filename=package://AiRobotURDF.SLDASM/meshes/steerBR.STL
- added link steerFL, mass 0.986568958091981; collision mesh filename=package://AiRobotURDF.SLDASM/meshes/steerFL.STL; visual mesh filename=package://AiRobotURDF.SLDASM/meshes/steerFL.STL
- added link steerFR, mass 0.98656895809198; collision mesh filename=package://AiRobotURDF.SLDASM/meshes/steerFR.STL; visual mesh filename=package://AiRobotURDF.SLDASM/meshes/steerFR.STL
- added link wheelBL, mass 0.764764182848667; collision mesh filename=package://AiRobotURDF.SLDASM/meshes/wheelBL.STL; visual mesh filename=package://AiRobotURDF.SLDASM/meshes/wheelBL.STL
- added link wheelBR, mass 0.764764182848667; collision mesh filename=package://AiRobotURDF.SLDASM/meshes/wheelBR.STL; visual mesh filename=package://AiRobotURDF.SLDASM/meshes/wheelBR.STL
- added link wheelFL, mass 0.764764182848668; collision mesh filename=package://AiRobotURDF.SLDASM/meshes/wheelFL.STL; visual mesh filename=package://AiRobotURDF.SLDASM/meshes/wheelFL.STL
- added link wheelFR, mass 0.764764182848667; collision mesh filename=package://AiRobotURDF.SLDASM/meshes/wheelFR.STL; visual mesh filename=package://AiRobotURDF.SLDASM/meshes/wheelFR.STL
- link base_link: mass 3.00064129669063 -> 6.94691712905856; geometry collision mesh filename=package://AiRobotURDF.SLDASM/meshes/base_link.STL; visual mesh filename=package://AiRobotURDF.SLDASM/meshes/base_link.STL
Joints:
- removed joint steer1
- removed joint steer2
- removed joint steer3
- removed joint steer4
- removed joint wheel1
- removed joint wheel2
- removed joint wheel3
- removed joint wheel4
- added joint steerBL: type fixed, parent base_link, child steerBL, origin xyz=0.0719999999999909 0.428000000000001 0.098 rpy=0 0 0, axis 0 0 0
- added joint steerBR: type fixed, parent base_link, child steerBR, origin xyz=0.071999999999999 0.0720000000000007 0.098 rpy=0 0 0, axis 0 0 0
- added joint steerFL: type fixed, parent base_link, child steerFL, origin xyz=0.427999999999993 0.428000000000008 0.098 rpy=0 0 3.14159265358979, axis 0 0 0
- added joint steerFR: type fixed, parent base_link, child steerFR, origin xyz=0.427999999999999 0.0720000000000044 0.098 rpy=0 0 3.14159265358979, axis 0 0 0
- added joint wheelBL: type fixed, parent steerBL, child wheelBL, origin xyz=0 0.0149999999999995 -0.056 rpy=1.5707963267949 1.5497746785967 0, axis 0 0 0
- added joint wheelBR: type fixed, parent steerBR, child wheelBR, origin xyz=0 0.015 -0.056 rpy=-1.5707963267949 -0.57401915441884 3.14159265358979, axis 0 0 0
- added joint wheelFL: type fixed, parent steerFL, child wheelFL, origin xyz=0 0.0150000000000002 -0.0559999999999995 rpy=-1.57079632679491 1.37893541128008 3.14159265358979, axis 0 0 0
- added joint wheelFR: type fixed, parent steerFR, child wheelFR, origin xyz=0 0.015 -0.0559999999999997 rpy=-1.57079632679489 -0.316982240676282 3.14159265358979, axis 0 0 0
