Commit message: urdf

File: URDF.urdf (robot description, URDF)
Before this commit: robot AiRobotURDF.SLDASM, 9 links, 8 joints
Links:
- link base_link: mass 6.94691712905856 -> 3.00064129669064; geometry collision mesh filename=package://URDF/meshes/base_link.STL; visual mesh filename=package://URDF/meshes/base_link.STL
- link steerBL: mass 0.98656895809198 -> 0.221804775243313; geometry collision mesh filename=package://URDF/meshes/steerBL.STL; visual mesh filename=package://URDF/meshes/steerBL.STL
- link steerBR: mass 0.98656895809198 -> 0.221804775243313; geometry collision mesh filename=package://URDF/meshes/steerBR.STL; visual mesh filename=package://URDF/meshes/steerBR.STL
- link steerFL: mass 0.986568958091981 -> 0.221804775243313; geometry collision mesh filename=package://URDF/meshes/steerFL.STL; visual mesh filename=package://URDF/meshes/steerFL.STL
- link steerFR: mass 0.98656895809198 -> 0.221804775243313; geometry collision mesh filename=package://URDF/meshes/steerFR.STL; visual mesh filename=package://URDF/meshes/steerFR.STL
- link wheelBL: geometry collision mesh filename=package://URDF/meshes/wheelBL.STL; visual mesh filename=package://URDF/meshes/wheelBL.STL
- link wheelBR: geometry collision mesh filename=package://URDF/meshes/wheelBR.STL; visual mesh filename=package://URDF/meshes/wheelBR.STL
- link wheelFL: geometry collision mesh filename=package://URDF/meshes/wheelFL.STL; visual mesh filename=package://URDF/meshes/wheelFL.STL
- link wheelFR: geometry collision mesh filename=package://URDF/meshes/wheelFR.STL; visual mesh filename=package://URDF/meshes/wheelFR.STL
Joints:
- joint wheelBL: axis 0 0 0 -> 0 0 1; origin xyz=0 0.0149999999999995 -0.056 rpy=1.5707963267949 1.5497746785967 0 -> xyz=0 0 -0.056 rpy=1.5707963267949 1.5497746785967 0; type fixed -> continuous
- joint wheelBR: axis 0 0 0 -> 0 0 1; origin xyz=0 0.015 -0.056 rpy=-1.5707963267949 -0.57401915441884 3.14159265358979 -> xyz=0 0 -0.056 rpy=-1.5707963267949 -0.57401915441884 3.14159265358979; type fixed -> continuous
- joint wheelFL: axis 0 0 0 -> 0 0 1; origin xyz=0 0.0150000000000002 -0.0559999999999995 rpy=-1.57079632679491 1.37893541128008 3.14159265358979 -> xyz=0 0 -0.056 rpy=-1.57079632679491 1.37893541128008 3.14159265358979; type fixed -> continuous
- joint wheelFR: axis 0 0 0 -> 0 0 1; origin xyz=0 0.015 -0.0559999999999997 rpy=-1.57079632679489 -0.316982240676282 3.14159265358979 -> xyz=0 0 -0.056 rpy=-1.57079632679489 -0.316982240676282 3.14159265358979; type fixed -> continuous
