Commit message: w

File: field/urdf/field.urdf (robot description, URDF)
Before this commit: robot field, 1 links, 0 joints
Links:
- added link box, mass 1.45641599999999; collision mesh filename=package://field/meshes/box.STL; visual mesh filename=package://field/meshes/box.STL
- added link wall, mass 78.9688883199999; collision mesh filename=package://field/meshes/wall.STL; visual mesh filename=package://field/meshes/wall.STL
- added link wall2, mass 15.15136; collision mesh filename=package://field/meshes/wall2.STL; visual mesh filename=package://field/meshes/wall2.STL
- added link wall3, mass 11.3635199999999; collision mesh filename=package://field/meshes/wall3.STL; visual mesh filename=package://field/meshes/wall3.STL
- link base_link: mass 248.19298432 -> 141.12
Joints:
- added joint box: type fixed, parent base_link, child box, origin xyz=-3.462 4.038 0 rpy=0 0 0, axis 0 0 0
- added joint wall: type fixed, parent base_link, child wall, origin xyz=0 0.01 0 rpy=0 0 0, axis 0 0 0
- added joint wall2: type fixed, parent base_link, child wall2, origin xyz=0 0.01 0 rpy=0 0 0, axis 0 0 0
- added joint wall3: type fixed, parent base_link, child wall3, origin xyz=0 0.01 0 rpy=0 0 0, axis 0 0 0
